File: PCB/ChocoBox/ChocoBox.kicad_sch (KiCad schematic)
At the start: 8 parts, among them J1 DTH22_01, J2 DTH22_02, J3 DS3231, J4 LCD2004A, J5 microSD, J6 Humidificador, J7 WaterLevel, U1 ESP32-DEVKIT-V1

Commit message: Inicio PCB
Parts:
- J4: footprint (none) -> Connector_PinSocket_2.54mm:PinSocket_1x04_P2.54mm_Vertical
- J5: footprint (none) -> Connector_PinSocket_2.54mm:PinSocket_1x06_P2.54mm_Vertical
- J7: footprint (none) -> Connector_PinSocket_2.54mm:PinSocket_1x03_P2.54mm_Vertical
Changed lines of the file:
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@@
       (effects (font (size 1.27 1.27)))
     )
-    (property "Footprint" "" (at 105.41 34.29 0)
+    (property "Footprint" "Connector_PinSocket_2.54mm:PinSocket_1x03_P2.54mm_Vertical" (at 105.41 34.29 0)
       (effects (font (size 1.27 1.27)) hide)
     )
@@
       (effects (font (size 1.27 1.27)))
     )
-    (property "Footprint" "" (at 21.59 68.58 0)
+    (property "Footprint" "Connector_PinSocket_2.54mm:PinSocket_1x06_P2.54mm_Vertical" (at 21.59 68.58 0)
       (effects (font (size 1.27 1.27)) hide)
     )
@@
       (effects (font (size 1.27 1.27)))
     )
-    (property "Footprint" "" (at 60.96 54.61 0)
-      (effects (font (size 1.27 1.27)) hide)
-    )
+    (property "Footprint" "Connector_PinSocket_2.54mm:PinSocket_1x04_P2.54mm_Vertical" (at 60.96 54.61 0)
+      (effects (font (size 1.27 1.27)) hide)
+    )

Commit message: PCB V1 Terminada
Parts:
- added J10: Vout-12V, Connector_PinSocket_2.54mm:PinSocket_1x02_P2.54mm_Vertical, symbol Connector_Generic:Conn_01x02
- added J11, J15, J16, J17, J18: Conn_01x01, Connector_PinSocket_2.54mm:PinSocket_1x01_P2.54mm_Vertical, symbol Connector_Generic:Conn_01x01
- added J12, J13: I2C, Connector_PinSocket_2.54mm:PinSocket_1x02_P2.54mm_Vertical, symbol Connector_Generic:Conn_01x02
- added J14: Vout-5V, Connector_PinSocket_2.54mm:PinSocket_1x02_P2.54mm_Vertical, symbol Connector_Generic:Conn_01x02
- added J8: Vin, TerminalBlock_Phoenix:TerminalBlock_Phoenix_MKDS-1,5-2-5.08_1x02_P5.08mm_Horizontal, symbol Connector:Screw_Terminal_01x02
- added J9: Calentador, Connector_PinSocket_2.54mm:PinSocket_1x02_P2.54mm_Vertical, symbol Connector_Generic:Conn_01x02
- added R1, R2: 10K, Resistor_THT:R_Axial_DIN0207_L6.3mm_D2.5mm_P10.16mm_Horizontal, symbol Device:R
- added SW1: BTN1, TerminalBlock_Phoenix:TerminalBlock_Phoenix_MKDS-1,5-2-5.08_1x02_P5.08mm_Horizontal, symbol Switch:SW_Push
- added SW2: BTN2, TerminalBlock_Phoenix:TerminalBlock_Phoenix_MKDS-1,5-2-5.08_1x02_P5.08mm_Horizontal, symbol Switch:SW_Push
- added U2: DCDC_StepDown_LM2596, Custom:YAAJ_DCDC_StepDown_LM2596, symbol StepDownLM2596:YAAJ_DCDC_StepDown_LM2596
Connections:
- net +3.3V: now also J17.1 (Pin_1), J18.1 (Pin_1), R1.1, R2.1
- net +5V: now also J11.1 (Pin_1), J14.2 (Pin_2), J15.1 (Pin_1), J16.1 (Pin_1), U2.4 (Vout); no longer U1.30 (VIN)
- net GND: now also J10.1 (Pin_1), J14.1 (Pin_1), J8.1 (Pin_1), SW1.2, SW2.2, U2.2 (GND), U2.3 (GND)
- net GPIO_SCL: now also J12.2 (Pin_2), J13.2 (Pin_2)
- net GPIO_SDA: now also J12.1 (Pin_1), J13.1 (Pin_1)
- net GPIO_35: now reaches U1.20 (D35)
- net GPIO_35: now also J9.2 (Pin_2)
- net BTN1: now reaches U1.26 (D14)
- net BTN1: now also R1.2, SW1.1
- net BTN2: now reaches U1.27 (D12)
- net BTN2: now also R2.2, SW2.1
- net RX2: now reaches U1.6 (RX2)
- net TX2: now reaches U1.7 (TX2)
- new net +12V: J10.2 (Pin_2), J8.2 (Pin_2), U2.1 (Vin)
- new net Vdrive: U1.30 (VIN)
- no-connect marks 3 -> 15
Other:
- note added: "Comunicaciones (Extra)"
- note added: "ESP32"
- note added: "Perifericos (Extra)"
- note added: "Potencia"

Commit message: PCB terminada
Parts:
- removed R2: 10K, Resistor_THT:R_Axial_DIN0207_L6.3mm_D2.5mm_P10.16mm_Horizontal, symbol Device:R
- removed SW2: BTN2, TerminalBlock_Phoenix:TerminalBlock_Phoenix_MKDS-1,5-2-5.08_1x02_P5.08mm_Horizontal, symbol Switch:SW_Push
- added J19: DS18B20-A, Connector_PinSocket_2.54mm:PinSocket_1x03_P2.54mm_Vertical, symbol Connector_Generic:Conn_01x03
- added J20: DS18B20-B, Connector_PinSocket_2.54mm:PinSocket_1x03_P2.54mm_Vertical, symbol Connector_Generic:Conn_01x03
- added J21: DS18B20-C, Connector_PinSocket_2.54mm:PinSocket_1x03_P2.54mm_Vertical, symbol Connector_Generic:Conn_01x03
- added J22: DS18B20-D, Connector_PinSocket_2.54mm:PinSocket_1x03_P2.54mm_Vertical, symbol Connector_Generic:Conn_01x03
- added R3: 4.7K, Resistor_THT:R_Axial_DIN0207_L6.3mm_D2.5mm_P10.16mm_Horizontal, symbol Device:R
- J14: value Vout-5V -> Vout-5V-Humidificador
- SW1: footprint TerminalBlock_Phoenix:TerminalBlock_Phoenix_MKDS-1,5-2-5.08_1x02_P5.08mm_Horizontal -> Connector_PinSocket_2.54mm:PinSocket_1x02_P2.54mm_Vertical
Connections:
- net +3.3V: now also J19.3 (Pin_3), J20.3 (Pin_3), J21.3 (Pin_3), J22.3 (Pin_3), R3.2
- net GND: now also J19.1 (Pin_1), J20.1 (Pin_1), J21.1 (Pin_1), J22.1 (Pin_1)
- net OneWire: now reaches U1.23 (D25)
- net OneWire: now also J19.2 (Pin_2), J20.2 (Pin_2), J21.2 (Pin_2), J22.2 (Pin_2), R3.1
- net BTN2: no longer names the net of U1.27 (D12)
- net RX2: no longer names the net of U1.6 (RX2)
- net TX2: no longer names the net of U1.7 (TX2)
- no-connect marks 15 -> 17
Other:
- note added: "OneWire (DS18B20)"
